File: HT485_DS/HT485_DS.kicad_sch (KiCad schematic)
At the start: 3 parts

Commit message: Fatta scheda sensore
Parts:
- J1: renamed from J?; footprint Connector_JST:JST_PH_S6B-PH-SM4-TB_1x06-1MP_P2.00mm_Horizontal -> Connector_JST:JST_PH_B6B-PH-K_1x06_P2.00mm_Vertical
- gave numbers to parts that had none: 2
Other:
- company: (none) -> RCF Srls
- title: (none) -> Digital Umidity Temperature Sensor over 485
Changed lines of the file:
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@@
 (kicad_sch (version 20211123) (generator eeschema)
   (paper "A4")
+  (title_block
+    (title "Digital Umidity Temperature Sensor over 485")
+    (date "2022-10-08")
+    (rev "1.0.0.0")
+    (company "RCF Srls")
+    (comment 1 "Luca Faccin")
+  )
   (junction (at 125.095 64.135) (diameter 0) (color 0 0 0 0)
   )
@@
   (symbol (lib_id "power:GND") (at 114.935 64.135 270) (mirror x) (unit 1)
     (in_bom yes) (on_board yes)
-    (property "Reference" "#PWR?" (id 0) (at 108.585 64.135 0)
+    (property "Reference" "#PWR03" (id 0) (at 108.585 64.135 0)
       (effects (font (size 1.27 1.27)) hide)
     )
@@
   (symbol (lib_id "power:GND") (at 105.41 81.28 270) (mirror x) (unit 1)
     (in_bom yes) (on_board yes)
-    (property "Reference" "#PWR?" (id 0) (at 99.06 81.28 0)
+    (property "Reference" "#PWR02" (id 0) (at 99.06 81.28 0)
       (effects (font (size 1.27 1.27)) hide)
     )
@@
   (symbol (lib_id "Connector:Conn_01x06_Female") (at 186.055 40.005 0) (unit 1)
     (in_bom yes) (on_board yes) (fields_autoplaced)
-    (property "Reference" "J?" (id 0) (at 187.96 40.0049 0)
+    (property "Reference" "J1" (id 0) (at 187.96 40.0049 0)
       (effects (font (size 1.27 1.27)) (justify left))
     )
@@
       (effects (font (size 1.27 1.27)) (justify left))
     )
-    (property "Footprint" "Connector_JST:JST_PH_S6B-PH-SM4-TB_1x06-1MP_P2.00mm_Horizontal" (id 2) (at 186.055 40.005 0)
+    (property "Footprint" "Connector_JST:JST_PH_B6B-PH-K_1x06_P2.00mm_Vertical" (id 2) (at 186.055 40.005 0)
       (effects (font (size 1.27 1.27)) hide)
     )
@@
   (symbol (lib_id "Sensor_Humidity:SHT31A-DIS") (at 125.095 78.74 0) (unit 1)
     (in_bom yes) (on_board yes) (fields_autoplaced)
-    (property "Reference" "U?" (id 0) (at 127.1144 68.58 0)
+    (property "Reference" "U1" (id 0) (at 127.1144 68.58 0)
       (effects (font (size 1.27 1.27)) (justify left))
     )
@@
   (symbol (lib_id "power:GND") (at 125.095 90.17 0) (mirror y) (unit 1)
     (in_bom yes) (on_board yes)
-    (property "Reference" "#PWR?" (id 0) (at 125.095 96.52 0)
+    (property "Reference" "#PWR05" (id 0) (at 125.095 96.52 0)
       (effects (font (size 1.27 1.27)) hide)
     )
@@
   (symbol (lib_id "power:GND") (at 167.005 47.625 270) (mirror x) (unit 1)
     (in_bom yes) (on_board yes)
-    (property "Reference" "#PWR?" (id 0) (at 160.655 47.625 0)
+    (property "Reference" "#PWR07" (id 0) (at 160.655 47.625 0)
       (effects (font (size 1.27 1.27)) hide)
     )
@@
   (symbol (lib_id "power:+3V3") (at 125.095 64.135 0) (unit 1)
     (in_bom yes) (on_board yes)
-    (property "Reference" "#PWR?" (id 0) (at 125.095 67.945 0)
+    (property "Reference" "#PWR04" (id 0) (at 125.095 67.945 0)
       (effects (font (size 1.27 1.27)) hide)
     )
@@
   (symbol (lib_id "power:GND") (at 105.41 76.2 270) (mirror x) (unit 1)
     (in_bom yes) (on_board yes)
-    (property "Reference" "#PWR?" (id 0) (at 99.06 76.2 0)
+    (property "Reference" "#PWR01" (id 0) (at 99.06 76.2 0)
       (effects (font (size 1.27 1.27)) hide)
     )
@@
   (symbol (lib_id "power:+3V3") (at 167.005 34.925 90) (unit 1)
     (in_bom yes) (on_board yes)
-    (property "Reference" "#PWR?" (id 0) (at 170.815 34.925 0)
+    (property "Reference" "#PWR06" (id 0) (at 170.815 34.925 0)
       (effects (font (size 1.27 1.27)) hide)
     )
@@
   (symbol (lib_id "Device:C_Small") (at 117.475 64.135 90) (unit 1)
     (in_bom yes) (on_board yes)
-    (property "Reference" "C?" (id 0) (at 114.935 68.58 0)
+    (property "Reference" "C1" (id 0) (at 114.935 68.58 0)
       (effects (font (size 1.27 1.27)) (justify left))
     )
@@
   )
   (symbol_instances
+    (path "/cf8dab28-2398-439b-8910-894e9189b574"
+      (reference "#PWR01") (unit 1) (value "GND") (footprint "")
+    )
+    (path "/08e80f4d-2315-4f23-b828-a20b6034c2a4"
+      (reference "#PWR02") (unit 1) (value "GND") (footprint "")
+    )
     (path "/03f49843-24c5-456e-ad6b-bcac91abf32b"
-      (reference "#PWR?") (unit 1) (value "GND") (footprint "")
-    )
-    (path "/08e80f4d-2315-4f23-b828-a20b6034c2a4"
-      (reference "#PWR?") (unit 1) (value "GND") (footprint "")
+      (reference "#PWR03") (unit 1) (value "GND") (footprint "")
+    )
+    (path "/b3252cf8-dd94-4db6-a9a7-350753bd1913"
+      (reference "#PWR04") (unit 1) (value "+3V3") (footprint "")
     )
     (path "/4f41dfd8-8d87-4bcc-9662-46132fb21c8c"
-      (reference "#PWR?") (unit 1) (value "GND") (footprint "")
+      (reference "#PWR05") (unit 1) (value "GND") (footprint "")
+    )
+    (path "/df6db40f-29ff-4073-9ed3-9c54e9ef4c92"
+      (reference "#PWR06") (unit 1) (value "+3V3") (footprint "")
     )
     (path "/9e5f17df-9355-4923-b26c-d7956244fcb1"
-      (reference "#PWR?") (unit 1) (value "GND") (footprint "")
-    )
-    (path "/b3252cf8-dd94-4db6-a9a7-350753bd1913"
-      (reference "#PWR?") (unit 1) (value "+3V3") (footprint "")
-    )
-    (path "/cf8dab28-2398-439b-8910-894e9189b574"
-      (reference "#PWR?") (unit 1) (value "GND") (footprint "")
-    )
-    (path "/df6db40f-29ff-4073-9ed3-9c54e9ef4c92"
-      (reference "#PWR?") (unit 1) (value "+3V3") (footprint "")
+      (reference "#PWR07") (unit 1) (value "GND") (footprint "")
     )
     (path "/f713eed1-d550-4808-9bcd-0068d047988a"
-      (reference "C?") (unit 1) (value "100nF") (footprint "Capacitor_SMD:C_0805_2012Metric")
+      (reference "C1") (unit 1) (value "100nF") (footprint "Capacitor_SMD:C_0805_2012Metric")
     )
     (path "/3b9709c1-8711-4f3f-9b84-45538d0df4e3"
-      (reference "J?") (unit 1) (value "H/T Sensor") (footprint "Connector_JST:JST_PH_S6B-PH-SM4-TB_1x06-1MP_P2.00mm_Horizontal")
+      (reference "J1") (unit 1) (value "H/T Sensor") (footprint "Connector_JST:JST_PH_B6B-PH-K_1x06_P2.00mm_Vertical")
     )
     (path "/4da6a415-d5b3-4c74-9e8c-aa9f9ea66912"
-      (reference "U?") (unit 1) (value "SHT31A-DIS") (footprint "Sensor_Humidity:Sensirion_DFN-8-1EP_2.5x2.5mm_P0.5mm_EP1.1x1.7mm")
-    )
-  )
+      (reference "U1") (unit 1) (value "SHT31A-DIS") (footprint "Sensor_Humidity:Sensirion_DFN-8-1EP_2.5x2.5mm_P0.5mm_EP1.1x1.7mm")
+    )
+  )
