File: HT_485.kicad_sch (KiCad schematic)
At the start: 114 parts, among them J1 485_1, J2 485_1, J3 PT1000, J4 H/T Sensor, J5 PRG, J6 PWR, Q1 BC817, Q10 BS170, Q2 BC817, Q3 BC817, Q4 BC817, Q5 BS170, Q6 BS170, Q7 BS170, Q8 BS170, Q9 BS170, SW1 485_PWR_1, SW2 485_PWR_2, U1 L7805, U2 TL082, U3 LD1086DT33TR, U4 ESP32-S3-WROOM-1U-N16R8, U5 LM2576S-12/NOPB, U7 TL431DBZ, U8 MAX485, U9 MAX485

Commit message: Aggiunto diodo per alimentazione CPU
Parts:
- added D16: 3.9V / 1W, Diode_SMD:D_SOD-128, symbol Device:D_Zener_Small
Connections:
- net +3V3: now also D16.1 (K)
- net GND: now also D16.2 (A)
Changed lines of the file:
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@@
   (junction (at 194.31 173.355) (diameter 0) (color 0 0 0 0)
   )
+  (junction (at 217.805 86.36) (diameter 0) (color 0 0 0 0)
+  )
   (junction (at 95.885 57.15) (diameter 0) (color 0 0 0 0)
   )
@@
     (stroke (width 0) (type default) (color 0 0 0 0))
   )
+  (wire (pts (xy 217.805 86.36) (xy 217.805 88.265))
+    (stroke (width 0) (type default) (color 0 0 0 0))
+  )
   (wire (pts (xy 125.095 199.39) (xy 125.095 203.835))
     (stroke (width 0) (type default) (color 0 0 0 0))
@@
     (stroke (width 0) (type default) (color 0 0 0 0))
   )
-  (wire (pts (xy 208.28 86.36) (xy 220.98 86.36))
+  (wire (pts (xy 208.28 86.36) (xy 217.805 86.36))
     (stroke (width 0) (type default) (color 0 0 0 0))
   )
@@
     (stroke (width 0) (type default) (color 0 0 0 0))
   )
+  (wire (pts (xy 217.805 86.36) (xy 220.98 86.36))
+    (stroke (width 0) (type default) (color 0 0 0 0))
+  )
   (wire (pts (xy 179.705 67.31) (xy 179.705 64.77))
     (stroke (width 0) (type default) (color 0 0 0 0))
@@
     (stroke (width 0) (type default) (color 0 0 0 0))
   )
+  (wire (pts (xy 217.805 93.345) (xy 217.805 95.25))
+    (stroke (width 0) (type default) (color 0 0 0 0))
+  )
   (wire (pts (xy 300.355 186.69) (xy 306.705 186.69))
     (stroke (width 0) (type default) (color 0 0 0 0))
@@
     (pin "1")
   )
+  (symbol (lib_id "power:GND") (at 217.805 95.25 0) (unit 1)
+    (in_bom yes) (on_board yes)
+    (property "Reference" "#PWR01" (id 0) (at 217.805 101.6 0)
+      (effects (font (size 1.27 1.27)) hide)
+    )
+    (property "Value" "GND" (id 1) (at 218.44 102.87 90)
+      (effects (font (size 1.27 1.27)) (justify left))
+    )
+    (property "Footprint" "" (id 2) (at 217.805 95.25 0)
+      (effects (font (size 1.27 1.27)) hide)
+    )
+    (property "Datasheet" "" (id 3) (at 217.805 95.25 0)
+      (effects (font (size 1.27 1.27)) hide)
+    )
+    (pin "1")
+  )
   (symbol (lib_id "power:GND") (at 133.985 132.715 0) (mirror y) (unit 1)
     (in_bom yes) (on_board yes) (fields_autoplaced)
@@
     (pin "8")
   )
+  (symbol (lib_id "Device:D_Zener_Small") (at 217.805 90.805 270) (unit 1)
+    (in_bom yes) (on_board yes)
+    (property "Reference" "D16" (id 0) (at 219.075 92.71 90)
+      (effects (font (size 1.27 1.27)) (justify left))
+    )
+    (property "Value" "3.9V / 1W" (id 1) (at 219.075 95.25 90)
+      (effects (font (size 1.27 1.27)) (justify left))
+    )
+    (property "Footprint" "Diode_SMD:D_SOD-128" (id 2) (at 217.805 90.805 90)
+      (effects (font (size 1.27 1.27)) hide)
+    )
+    (property "Datasheet" "~" (id 3) (at 217.805 90.805 90)
+      (effects (font (size 1.27 1.27)) hide)
+    )
+    (pin "1")
+    (pin "2")
+  )
   (symbol (lib_id "Device:R_Small") (at 63.5 132.715 270) (unit 1)
     (in_bom yes) (on_board yes)
@@
   )
   (symbol_instances
+    (path "/b1b48d6c-3e44-4cb8-8411-0aa616ca78b3"
+      (reference "#PWR01") (unit 1) (value "GND") (footprint "")
+    )
     (path "/8302af2c-d18b-4f4f-9075-36f3eaee599a"
       (reference "#PWR02") (unit 1) (value "+12V") (footprint "")
@@
       (reference "D15") (unit 1) (value "VSSAF522-M3/H") (footprint "Diode_SMD:D_SMA-SMB_Universal_Handsoldering")
     )
+    (path "/c963d997-e95a-421a-b6f0-60029dfd5d48"
+      (reference "D16") (unit 1) (value "3.9V / 1W") (footprint "Diode_SMD:D_SOD-128")
+    )
     (path "/cfb45fe0-353a-40a9-8b84-c83bb6901246"

Commit message: Correto mosfet voltage shifter.
Parts:
- removed Q10, Q5, Q6, Q7, Q8, Q9: BS170, Package_TO_SOT_SMD:SOT-23, symbol Transistor_FET:BS170
- added Q10, Q5, Q6, Q7, Q8, Q9: Si2302CDS, Package_TO_SOT_SMD:SOT-23, symbol Device:Q_NMOS_GSD
- R12: value 1K 1% -> 560R 1%
Connections:
- net +3V3: now also Q10.1 (G), Q5.1 (G), Q6.1 (G), Q7.1 (G), Q8.1 (G), Q9.1 (G)
- net DEH1: now also Q7.3 (D)
- net DEH2: now also Q10.3 (D)
- net RXH1: now also Q5.3 (D)
- net RXH2: now also Q8.3 (D)
- net TXH1: now also Q6.3 (D)
- net TXH2: now also Q9.3 (D)
- net at R21.1, R32.1: now also Q5.2 (S)
- net at R38.1, R41.1: now also Q8.2 (S)
- net at R39.1, R42.1: now also Q9.2 (S)
- net at R23.1, R33.1: now also Q6.2 (S)
- net at R40.1, R43.1: now also Q10.2 (S)
- net at R31.1, R34.1: now also Q7.2 (S)
- net -12V renamed -10V

Commit message: Revisionato master
Parts:
- J6: footprint TerminalBlock_Phoenix:TerminalBlock_Phoenix_PT-1,5-2-3.5-H_1x02_P3.50mm_Horizontal -> TerminalBlock_Phoenix:TerminalBlock_Phoenix_PT-1,5-2-5.0-H_1x02_P5.00mm_Horizontal
Connections:
- net ALERT: now also U4.38 (GPIO2/TOUCH2/ADC1_CH1); no longer U4.35 (MTMS/GPIO42)
- net DE1: now also U4.17 (GPIO9/TOUCH9/ADC1_CH8/FSPIHD/SUBSPIHD); no longer U4.18 (GPIO10/TOUCH10/ADC1_CH9/FSPICS0/FSPIIO4/SUBSPICS0)
- net RESET: now also U4.35 (MTMS/GPIO42); no longer U4.38 (GPIO2/TOUCH2/ADC1_CH1)
- net RX1: now also U4.15 (GPIO3/TOUCH3/ADC1_CH2); no longer U4.17 (GPIO9/TOUCH9/ADC1_CH8/FSPIHD/SUBSPIHD)
- net RX2: now also U4.20 (GPIO12/TOUCH11/ADC2_CH0/FSPICS0/FSPIIO4/SUBSPICS0); no longer U4.22 (GPIO14/TOUCH14/ADC2_CH3/FSPIWP/FSPIDQS/SUBSPIWP)
- net SCL: now also U4.33 (MTDO/GPIO40/CLK_OUT2); no longer U4.34 (MTDI/GPIO41/CLK_OUT1)
- net SDA: now also U4.34 (MTDI/GPIO41/CLK_OUT1); no longer U4.33 (MTDO/GPIO40/CLK_OUT2)
- net TX1: now also U4.18 (GPIO10/TOUCH10/ADC1_CH9/FSPICS0/FSPIIO4/SUBSPICS0); no longer U4.15 (GPIO3/TOUCH3/ADC1_CH2)
- net TX2: now also U4.22 (GPIO14/TOUCH14/ADC2_CH3/FSPIWP/FSPIDQS/SUBSPIWP); no longer U4.20 (GPIO12/TOUCH11/ADC2_CH0/FSPICS0/FSPIIO4/SUBSPICS0)
- no-connect marks 13 -> 20
Changed lines of the file:
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@@
   (junction (at 363.855 119.38) (diameter 0) (color 0 0 0 0)
   )
+  (no_connect (at 220.98 40.64))
+  (no_connect (at 220.98 43.18))
+  (no_connect (at 220.98 71.12))
+  (no_connect (at 220.98 73.66))
   (no_connect (at 339.09 62.23))
+  (no_connect (at 220.98 76.2))
+  (no_connect (at 339.09 49.53))
+  (no_connect (at 339.09 52.07))
   (no_connect (at 339.09 59.69))
   (no_connect (at 339.09 57.15))
@@
     (effects (font (size 1.27 1.27)) (justify left bottom))
   )
-  (label "DE1" (at 208.915 55.88 0)
-    (effects (font (size 1.27 1.27)) (justify left bottom))
-  )
   (label "TX1" (at 177.8 159.385 0)
     (effects (font (size 1.27 1.27)) (justify left bottom))
@@
     (effects (font (size 1.27 1.27)) (justify left bottom))
   )
+  (label "TX2" (at 208.915 66.04 0)
+    (effects (font (size 1.27 1.27)) (justify left bottom))
+  )
   (label "SCL" (at 379.73 44.45 0)
     (effects (font (size 1.27 1.27)) (justify left bottom))
@@
     (effects (font (size 1.27 1.27)) (justify right bottom))
   )
-  (label "TX1" (at 208.915 38.1 0)
-    (effects (font (size 1.27 1.27)) (justify left bottom))
-  )
   (label "RXH1" (at 342.265 132.08 0)
     (effects (font (size 1.27 1.27)) (justify left bottom))
@@
     (effects (font (size 1.27 1.27)) (justify right bottom))
   )
-  (label "TX2" (at 208.915 60.96 0)
-    (effects (font (size 1.27 1.27)) (justify left bottom))
-  )
   (label "TXH1" (at 226.06 159.385 180)
     (effects (font (size 1.27 1.27)) (justify right bottom))
@@
     (effects (font (size 1.27 1.27)) (justify left bottom))
   )
-  (label "RX1" (at 208.915 53.34 0)
-    (effects (font (size 1.27 1.27)) (justify left bottom))
-  )
   (label "RXH2" (at 312.42 129.54 180)
     (effects (font (size 1.27 1.27)) (justify right bottom))
@@
     (effects (font (size 1.27 1.27)) (justify right bottom))
   )
-  (label "RX2" (at 208.915 66.04 0)
-    (effects (font (size 1.27 1.27)) (justify left bottom))
-  )
   (label "PT1000_ADC" (at 207.01 33.02 0)
     (effects (font (size 1.27 1.27)) (justify left bottom))
@@
     (effects (font (size 1.27 1.27)) (justify right bottom))
   )
+  (label "ALERT" (at 207.01 35.56 0)
+    (effects (font (size 1.27 1.27)) (justify left bottom))
+  )
   (label "TXH2" (at 340.995 186.69 0)
     (effects (font (size 1.27 1.27)) (justify left bottom))
@@
     (effects (font (size 1.27 1.27)) (justify left bottom))
   )
-  (label "SDA" (at 351.79 72.39 180)
-    (effects (font (size 1.27 1.27)) (justify right bottom))
-  )
   (label "DE1" (at 177.8 187.325 0)
     (effects (font (size 1.27 1.27)) (justify left bottom))
   )
-  (label "RESET" (at 207.01 35.56 0)
-    (effects (font (size 1.27 1.27)) (justify left bottom))
+  (label "RESET" (at 353.06 77.47 180)
+    (effects (font (size 1.27 1.27)) (justify right bottom))
   )
   (label "DEH1" (at 342.265 134.62 0)
@@
     (effects (font (size 1.27 1.27)) (justify left bottom))
   )
-  (label "SCL" (at 351.79 74.93 180)
+  (label "SDA" (at 351.79 74.93 180)
     (effects (font (size 1.27 1.27)) (justify right bottom))
   )
+  (label "DE1" (at 208.915 53.34 0)
+    (effects (font (size 1.27 1.27)) (justify left bottom))
+  )
+  (label "RX2" (at 208.915 60.96 0)
+    (effects (font (size 1.27 1.27)) (justify left bottom))
+  )
   (label "VCC2" (at 306.705 170.18 270)
     (effects (font (size 1.27 1.27)) (justify right bottom))
@@
     (effects (font (size 1.27 1.27)) (justify right bottom))
   )
-  (label "ALERT" (at 353.06 77.47 180)
-    (effects (font (size 1.27 1.27)) (justify right bottom))
-  )
   (label "U0TXD" (at 370.205 26.67 0)
     (effects (font (size 1.27 1.27)) (justify left bottom))
@@
     (effects (font (size 1.27 1.27)) (justify right bottom))
   )
+  (label "RX1" (at 208.915 38.1 0)
+    (effects (font (size 1.27 1.27)) (justify left bottom))
+  )
   (label "TXH1" (at 342.265 139.7 0)
     (effects (font (size 1.27 1.27)) (justify left bottom))
   )
+  (label "TX1" (at 208.915 55.88 0)
+    (effects (font (size 1.27 1.27)) (justify left bottom))
+  )
   (label "485_2-" (at 372.745 186.69 0)
     (effects (font (size 1.27 1.27)) (justify left bottom))
@@
     (effects (font (size 1.27 1.27)) (justify left bottom))
   )
+  (label "SCL" (at 351.79 72.39 180)
+    (effects (font (size 1.27 1.27)) (justify right bottom))
+  )
   (label "DEH2" (at 340.995 181.61 0)
     (effects (font (size 1.27 1.27)) (justify left bottom))
@@
       (effects (font (size 1.27 1.27)) (justify left))
     )
-    (property "Footprint" "TerminalBlock_Phoenix:TerminalBlock_Phoenix_PT-1,5-2-3.5-H_1x02_P3.50mm_Horizontal" (id 2) (at 125.73 17.78 0)
+    (property "Footprint" "TerminalBlock_Phoenix:TerminalBlock_Phoenix_PT-1,5-2-5.0-H_1x02_P5.00mm_Horizontal" (id 2) (at 125.73 17.78 0)
       (effects (font (size 1.27 1.27)) hide)
     )
@@
     )
     (path "/57c32ce9-6606-479d-bbf1-7cf360aed045"
-      (reference "J6") (unit 1) (value "PWR") (footprint "TerminalBlock_Phoenix:TerminalBlock_Phoenix_PT-1,5-2-3.5-H_1x02_P3.50mm_Horizontal")
+      (reference "J6") (unit 1) (value "PWR") (footprint "TerminalBlock_Phoenix:TerminalBlock_Phoenix_PT-1,5-2-5.0-H_1x02_P5.00mm_Horizontal")
     )
     (path "/3af9e07a-b539-465e-b8d3-40cd261f557a"
