File: HT_485.kicad_sch (KiCad schematic)
At the start: 115 parts, among them J1 485_1, J2 485_1, J3 PT1000, J4 H/T Sensor, J5 PRG, J6 PWR, Q1 BC817, Q10 Si2302CDS, Q2 BC817, Q3 BC817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

Commit message: Aggiunti logo MME. Versione 1.0.1.0
Parts:
- added H1, H2: MountingHole, MountingHole:MountingHole_3.2mm_M3, symbol Mechanical:MountingHole
Other:
- company: RCF Srls -> MecMan Engineering SRL
- title: Umidity Temperature Sensor over 485 -> HT 485
Changed lines of the file:
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@@
   (paper "A3")
   (title_block
-    (title "Umidity Temperature Sensor over 485")
-    (date "2022-07-07")
+    (title "HT 485")
+    (date "2022-10-22")
     (rev "1.0.1.0")
-    (company "RCF Srls")
+    (company "MecMan Engineering SRL")
     (comment 1 "Luca Faccin")
   )
@@
   (no_connect (at 339.09 62.23))
   (no_connect (at 220.98 76.2))
-  (no_connect (at 339.09 49.53))
   (no_connect (at 339.09 52.07))
+  (no_connect (at 339.09 49.53))
   (no_connect (at 339.09 59.69))
   (no_connect (at 339.09 57.15))
@@
     (pin "3")
   )
+  (symbol (lib_id "Mechanical:MountingHole") (at 163.83 234.95 0) (unit 1)
+    (in_bom yes) (on_board yes) (fields_autoplaced)
+    (property "Reference" "H1" (id 0) (at 166.37 233.6799 0)
+      (effects (font (size 1.27 1.27)) (justify left))
+    )
+    (property "Value" "MountingHole" (id 1) (at 166.37 236.2199 0)
+      (effects (font (size 1.27 1.27)) (justify left))
+    )
+    (property "Footprint" "MountingHole:MountingHole_3.2mm_M3" (id 2) (at 163.83 234.95 0)
+      (effects (font (size 1.27 1.27)) hide)
+    )
+    (property "Datasheet" "~" (id 3) (at 163.83 234.95 0)
+      (effects (font (size 1.27 1.27)) hide)
+    )
+  )
   (symbol (lib_id "power:GND") (at 360.045 110.49 0) (mirror x) (unit 1)
     (in_bom yes) (on_board yes) (fields_autoplaced)
@@
     (pin "2")
   )
+  (symbol (lib_id "Mechanical:MountingHole") (at 163.83 242.57 0) (unit 1)
+    (in_bom yes) (on_board yes) (fields_autoplaced)
+    (property "Reference" "H2" (id 0) (at 166.37 241.2999 0)
+      (effects (font (size 1.27 1.27)) (justify left))
+    )
+    (property "Value" "MountingHole" (id 1) (at 166.37 243.8399 0)
+      (effects (font (size 1.27 1.27)) (justify left))
+    )
+    (property "Footprint" "MountingHole:MountingHole_3.2mm_M3" (id 2) (at 163.83 242.57 0)
+      (effects (font (size 1.27 1.27)) hide)
+    )
+    (property "Datasheet" "~" (id 3) (at 163.83 242.57 0)
+      (effects (font (size 1.27 1.27)) hide)
+    )
+  )
   (symbol (lib_id "power:GND") (at 83.82 73.66 0) (unit 1)
     (in_bom yes) (on_board yes)
@@
       (reference "D16") (unit 1) (value "3.9V / 1W") (footprint "Diode_SMD:D_SOD-128")
     )
+    (path "/435f79ee-27a2-427d-9473-883032d067f5"
+      (reference "H1") (unit 1) (value "MountingHole") (footprint "MountingHole:MountingHole_3.2mm_M3")
+    )
+    (path "/c3d6f923-fdcc-4592-966d-ddded5f8a0da"
+      (reference "H2") (unit 1) (value "MountingHole") (footprint "MountingHole:MountingHole_3.2mm_M3")
+    )
     (path "/cfb45fe0-353a-40a9-8b84-c83bb6901246"

Commit message: Messi connettori 485 a passo 5. Aggiornata versione a 1.0.1.1
Parts:
- J1, J2: footprint TerminalBlock_Phoenix:TerminalBlock_Phoenix_PT-1,5-2-3.5-H_1x02_P3.50mm_Horizontal -> TerminalBlock_Phoenix:TerminalBlock_Phoenix_PT-1,5-2-5.0-H_1x02_P5.00mm_Horizontal
